File: STM32_DEV.kicad_sch (KiCad schematic)
At the start: 13 parts

Commit message: sch and pcb files udpated
Parts:
- added C1, C2: 10p, Capacitor_SMD:C_0402_1005Metric, symbol Device:C
- added C12, C13: 22u, Capacitor_SMD:C_0805_2012Metric, symbol Device:C
- added D1: RED, LED_SMD:LED_0603_1608Metric, symbol Device:LED
- added H1, H2: MountingHole, MountingHole:MountingHole_2.2mm_M2, symbol Mechanical:MountingHole
- added J1, J3, J5: Conn_01x04_Male, Connector_PinHeader_2.54mm:PinHeader_1x04_P2.54mm_Vertical, symbol Connector:Conn_01x04_Male
- added J2: Conn_01x06_Male, Connector_PinHeader_2.54mm:PinHeader_1x06_P2.54mm_Vertical, symbol Connector:Conn_01x06_Male
- added J4: USB_B_Micro, Connector_USB:USB_Micro-B_Wuerth_629105150521, symbol Connector:USB_B_Micro
- added R1, R2, R4, R5: 1k5, Resistor_SMD:R_0402_1005Metric, symbol Device:R
- added U2: AMS1117-3.3, Package_TO_SOT_SMD:SOT-223-3_TabPin2, symbol Regulator_Linear:AMS1117-3.3
- added Y1: 16MHz, Crystal:Crystal_SMD_3225-4Pin_3.2x2.5mm, symbol Device:Crystal_GND24
- C10, C11, C4, C5, C6, C7, C8, C9: renamed from C?; footprint (none) -> Capacitor_SMD:C_0402_1005Metric
- C3: renamed from C?; footprint (none) -> Capacitor_SMD:C_0603_1608Metric
- FB1: renamed from FB?; footprint (none) -> Inductor_SMD:L_0603_1608Metric
- R3: renamed from R?; footprint (none) -> Resistor_SMD:R_0402_1005Metric
- SW1: renamed from SW?; footprint (none) -> Button_Switch_SMD:SW_SPDT_PCM12
- gave numbers to parts that had none: 1
Connections:
- net +3V3: now also C13.1, D1.2 (A), J1.1 (Pin_1), J2.1 (Pin_1), J3.1 (Pin_1), J5.1 (Pin_1), R1.1, R2.1, R4.1, U2.2 (VO)
- net GND: now also C1.2, C12.2, C13.2, C2.2, J1.4 (Pin_4), J2.6 (Pin_6), J3.4 (Pin_4), J4.5 (GND), J5.4 (Pin_4), R5.2, U2.1 (GND), Y1.2, Y1.4
- net PA0: now reaches U1.10 (PA0)
- net PA1: now reaches U1.11 (PA1)
- net PA2: now reaches U1.12 (PA2)
- net PA3: now reaches U1.13 (PA3)
- net PA4: now reaches U1.14 (PA4)
- net SPI1_SCK: now reaches U1.15 (PA5)
- net SPI1_SCK: now also J2.2 (Pin_2)
- net SPI1_MISO: now reaches U1.16 (PA6)
- net SPI1_MISO: now also J2.3 (Pin_3)
- net SPI1_MOSI: now reaches U1.17 (PA7)
- net SPI1_MOSI: now also J2.4 (Pin_4)
- net ~CS: now reaches U1.18 (PB0)
- net ~CS: now also J2.5 (Pin_5)
- net PB1: now reaches U1.19 (PB1)
- net PC13: now reaches U1.2 (PC13)
- net PB2: now reaches U1.20 (PB2)
- net I2C2_SCL: now reaches U1.21 (PB10)
- net I2C2_SCL: now also J1.2 (Pin_2), R1.2
- net I2C2_SDA: now reaches U1.22 (PB11)
- net I2C2_SDA: now also J1.3 (Pin_3), R2.2
- net PB12: now reaches U1.25 (PB12)
- net PB13: now reaches U1.26 (PB13)
- net PB14: now reaches U1.27 (PB14)
- net PB15: now reaches U1.28 (PB15)
- net PA8: now reaches U1.29 (PA8)
- net PC14: now reaches U1.3 (PC14)
- net PA9: now reaches U1.30 (PA9)
- net PA10: now reaches U1.31 (PA10)
- net USB_D-: now reaches U1.32 (PA11)
- net USB_D-: now also J4.2 (D-)
- net USB_D+: now reaches U1.33 (PA12)
- net USB_D+: now also J4.3 (D+), R4.2
- net SWD_IO: now reaches U1.34 (PA13)
- net SWD_IO: now also J5.2 (Pin_2)
- net SW_CLK: now reaches U1.37 (PA14)
- net SW_CLK: now also J5.3 (Pin_3)
- net PA15: now reaches U1.38 (PA15)
- net PB3: now reaches U1.39 (PB3)
- net PC15: now reaches U1.4 (PC15)
- net PB4: now reaches U1.40 (PB4)
- net PB5: now reaches U1.41 (PB5)
- net USART1_TX: now reaches U1.42 (PB6)
- net USART1_TX: now also J3.2 (Pin_2)
- net USART1_RX: now reaches U1.43 (PB7)
- net USART1_RX: now also J3.3 (Pin_3)
- net PB8: now reaches U1.45 (PB8)
- net PB9: now reaches U1.46 (PB9)
- net HSE_IN: now reaches U1.5 (PD0)
- net HSE_IN: now also C1.1, Y1.1
- net HSE_OUT: now reaches U1.6 (PD1)
- net HSE_OUT: now also C2.1, Y1.3
- new net PWR_LED_K: D1.1 (K), R5.1
- new net VBUS: C12.1, J4.1 (VBUS), U2.3 (VI)
- no-connect marks 0 -> 2
Other:
- note added: "Crystal Oscillator design: 2 ext load Caps. 1 omitted feed resistance, maybe of need to limit distortion & overdriving the crystal"
- note added: "Need USB+ pulled up to get detected"
- note added: "PULL UP FOR I2C BUS"
- note added: "SWD CONNECTOR"
- note added: "Sheild left floating. ID pin only used while USB On-The-Go. VBUS is the Voltage feed to the regulator"
- company: (none) -> @SKrish_K
- title: (none) -> STM32_DEV_BOARD
- moved on the sheet: C10, C11, C3, C4, C5, C6, C7, C8, C9, FB1, R3, SW1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
